Commit message: Panda arm simulation working

File: install/franka_moveit_config/share/franka_moveit_config/config/hand.xacro (robot description, xacro)
@@ -1,23 +1 @@
-<?xml version="1.0" ?>
-<robot xmlns:xacro="http://www.ros.org/wiki/xacro" name="panda">
-  <xacro:macro name="hand">
-    <!--GROUPS: Representation of a set of joints and links. This can be useful for specifying DOF to plan for, defining arms, end effectors, etc-->
-    <!--LINKS: When a link is specified, the parent joint of that link (if it exists) is automatically included-->
-    <!--JOINTS: When a joint is specified, the child link of that joint (which will always exist) is automatically included-->
-    <!--CHAINS: When a chain is specified, all the links along the chain (including endpoints) are included in the group. Additionally, all the joints that are parents to included links are also included. This means that joints along the chain and the parent joint of the base link are included in the group-->
-    <!--SUBGROUPS: Groups can also be formed by referencing to already defined group names-->
-    <group name="hand">
-      <link name="panda_hand" />
-      <link name="panda_leftfinger" />
-      <link name="panda_rightfinger" />
-      <joint name="panda_finger_joint1" />
-      <passive_joint name="panda_finger_joint2" />
-    </group>
-    <!--GROUP STATES: Purpose: Define a named state for a particular group, in terms of joint values. This is useful to define states like 'folded arms'-->
-    <!--END EFFECTOR: Purpose: Represent information about an end effector.-->
-    <!--DISABLE COLLISIONS: By default it is assumed that any link of the robot could potentially come into collision with any other link in the robot. This tag disables collision checking between a specified pair of links. -->
-    <disable_collisions link1="panda_hand" link2="panda_leftfinger" reason="Adjacent" />
-    <disable_collisions link1="panda_hand" link2="panda_rightfinger" reason="Adjacent" />
-    <disable_collisions link1="panda_leftfinger" link2="panda_rightfinger" reason="Default" />
-  </xacro:macro>
-</robot>
+/home/merlabros2/RBE595/src/franka_moveit_config/config/hand.xacro

File: install/franka_moveit_config/share/franka_moveit_config/config/panda.ros2_control.xacro (robot description, xacro)
@@ -1,78 +1 @@
-<?xml version="1.0"?>
-<robot xmlns:xacro="http://www.ros.org/wiki/xacro">
-    <xacro:macro name="panda_ros2_control" params="name initial_positions_file">
-        <xacro:property name="initial_positions" value="${load_yaml(initial_positions_file)['initial_positions']}"/>
-        <ros2_control name="${name}" type="system">
-            <hardware>
-                <!-- By default, set up controllers for simulation. This won't work on real hardware -->
-                <plugin>mock_components/GenericSystem</plugin>
-                <!-- <plugin>franka_hardware/FrankaHardwareInterface</plugin> -->
-                <!-- <param name="robot_ip">172.16.0.2</param> -->
-            </hardware>
-            <joint name="panda_joint1">
-                <command_interface name="position"/>
-                <command_interface name="velocity"/>
-                <state_interface name="position">
-                  <param name="initial_value">${initial_positions['panda_joint1']}</param>
-                </state_interface>
-                <state_interface name="velocity"/>
-            </joint>
-            <joint name="panda_joint2">
-                <command_interface name="position"/>
-                <command_interface name="velocity"/>
-                <state_interface name="position">
-                  <param name="initial_value">${initial_positions['panda_joint2']}</param>
-                </state_interface>
-                <state_interface name="velocity"/>
-            </joint>
-            <joint name="panda_joint3">
-                <command_interface name="position"/>
-                <command_interface name="velocity"/>
-                <state_interface name="position">
-                  <param name="initial_value">${initial_positions['panda_joint3']}</param>
-                </state_interface>
-                <state_interface name="velocity"/>
-            </joint>
-            <joint name="panda_joint4">
-                <command_interface name="position"/>
-                <command_interface name="velocity"/>
-                <state_interface name="position">
-                  <param name="initial_value">${initial_positions['panda_joint4']}</param>
-                </state_interface>
-                <state_interface name="velocity"/>
-            </joint>
-            <joint name="panda_joint5">
-                <command_interface name="position"/>
-                <command_interface name="velocity"/>
-                <state_interface name="position">
-                  <param name="initial_value">${initial_positions['panda_joint5']}</param>
-                </state_interface>
-                <state_interface name="velocity"/>
-            </joint>
-            <joint name="panda_joint6">
-                <command_interface name="position"/>
-                <command_interface name="velocity"/>
-                <state_interface name="position">
-                  <param name="initial_value">${initial_positions['panda_joint6']}</param>
-                </state_interface>
-                <state_interface name="velocity"/>
-            </joint>
-            <joint name="panda_joint7">
-                <command_interface name="position"/>
-                <command_interface name="velocity"/>
-                <state_interface name="position">
-                  <param name="initial_value">${initial_positions['panda_joint7']}</param>
-                </state_interface>
-                <state_interface name="velocity"/>
-            </joint>
-            <joint name="panda_finger_joint1">
-                <command_interface name="position"/>
-                <command_interface name="velocity"/>
-                <state_interface name="position">
-                  <param name="initial_value">${initial_positions['panda_finger_joint1']}</param>
-                </state_interface>
-                <state_interface name="velocity"/>
-            </joint>
-        </ros2_control>
-    </xacro:macro>
-</robot>
+/home/merlabros2/RBE595/src/franka_moveit_config/config/panda.ros2_control.xacro

File: install/franka_moveit_config/share/franka_moveit_config/config/panda.urdf.xacro (robot description, xacro)
@@ -1,9 +1 @@
-<?xml version="1.0"?>
-<robot xmlns:xacro="http://www.ros.org/wiki/xacro" name="panda">
-    <xacro:arg name="initial_positions_file" default="initial_positions.yaml" />
-    <!-- Import panda urdf file -->
-    <xacro:include filename="$(find moveit_resources_panda_description)/urdf/panda.urdf" />
-    <!-- Import control_xacro -->
-    <xacro:include filename="panda.ros2_control.xacro" />
-    <xacro:panda_ros2_control name="FakeSystem" initial_positions_file="$(arg initial_positions_file)"/>
-</robot>
+/home/merlabros2/RBE595/src/franka_moveit_config/config/panda.urdf.xacro

File: install/franka_moveit_config/share/franka_moveit_config/config/panda_arm.srdf.xacro (robot description, xacro)
@@ -1,9 +1 @@
-<?xml version='1.0' encoding='utf-8'?>
-<!--This does not replace URDF, and is not an extension of URDF.
-    This is a format for representing semantic information about the robot structure.
-    A URDF file must exist for this robot as well, where the joints and the links that are referenced are defined
--->
-<robot xmlns:xacro="http://www.ros.org/wiki/xacro" name="panda">
-  <xacro:include filename="$(find moveit_resources_panda_moveit_config)/config/panda_arm.xacro" />
-  <xacro:panda_arm />
-</robot>
+/home/merlabros2/RBE595/src/franka_moveit_config/config/panda_arm.srdf.xacro

File: install/franka_moveit_config/share/franka_moveit_config/config/panda_arm.xacro (robot description, xacro)
@@ -1,64 +1 @@
-<?xml version="1.0" ?>
-<robot xmlns:xacro="http://www.ros.org/wiki/xacro" name="panda">
-  <xacro:macro name="panda_arm">
-    <!--GROUPS: Representation of a set of joints and links. This can be useful for specifying DOF to plan for, defining arms, end effectors, etc-->
-    <!--LINKS: When a link is specified, the parent joint of that link (if it exists) is automatically included-->
-    <!--JOINTS: When a joint is specified, the child link of that joint (which will always exist) is automatically included-->
-    <!--CHAINS: When a chain is specified, all the links along the chain (including endpoints) are included in the group. Additionally, all the joints that are parents to included links are also included. This means that joints along the chain and the parent joint of the base link are included in the group-->
-    <!--SUBGROUPS: Groups can also be formed by referencing to already defined group names-->
-    <group name="panda_arm">
-      <chain base_link="panda_link0" tip_link="panda_link8" />
-    </group>
-    <!--GROUP STATES: Purpose: Define a named state for a particular group, in terms of joint values. This is useful to define states like 'folded arms'-->
-    <group_state name="ready" group="panda_arm">
-      <joint name="panda_joint1" value="0" />
-      <joint name="panda_joint2" value="-0.785" />
-      <joint name="panda_joint3" value="0" />
-      <joint name="panda_joint4" value="-2.356" />
-      <joint name="panda_joint5" value="0" />
-      <joint name="panda_joint6" value="1.571" />
-      <joint name="panda_joint7" value="0.785" />
-    </group_state>
-    <group_state name="extended" group="panda_arm">
-      <joint name="panda_joint1" value="0" />
-      <joint name="panda_joint2" value="0" />
-      <joint name="panda_joint3" value="0" />
-      <joint name="panda_joint4" value="0" />
-      <joint name="panda_joint5" value="0" />
-      <joint name="panda_joint6" value="1.571" />
-      <joint name="panda_joint7" value="0.785" />
-    </group_state>
-    <group_state name="transport" group="panda_arm">
-      <joint name="panda_joint1" value="0" />
-      <joint name="panda_joint2" value="-0.5599" />
-      <joint name="panda_joint3" value="0" />
-      <joint name="panda_joint4" value="-2.97" />
-      <joint name="panda_joint5" value="0" />
-      <joint name="panda_joint6" value="0" />
-      <joint name="panda_joint7" value="0.785" />
-    </group_state>
-    <!--END EFFECTOR: Purpose: Represent information about an end effector.-->
-    <!--VIRTUAL JOINT: Purpose: this element defines a virtual joint between a robot link and an external frame of reference (considered fixed with respect to the robot)-->
-    <virtual_joint name="virtual_joint" type="floating" parent_frame="world" child_link="panda_link0" />
-    <!--DISABLE COLLISIONS: By default it is assumed that any link of the robot could potentially come into collision with any other link in the robot. This tag disables collision checking between a specified pair of links. -->
-    <disable_collisions link1="panda_link0" link2="panda_link1" reason="Adjacent" />
-    <disable_collisions link1="panda_link0" link2="panda_link2" reason="Never" />
-    <disable_collisions link1="panda_link0" link2="panda_link3" reason="Never" />
-    <disable_collisions link1="panda_link0" link2="panda_link4" reason="Never" />
-    <disable_collisions link1="panda_link1" link2="panda_link2" reason="Adjacent" />
-    <disable_collisions link1="panda_link1" link2="panda_link3" reason="Never" />
-    <disable_collisions link1="panda_link1" link2="panda_link4" reason="Never" />
-    <disable_collisions link1="panda_link2" link2="panda_link3" reason="Adjacent" />
-    <disable_collisions link1="panda_link2" link2="panda_link4" reason="Never" />
-    <disable_collisions link1="panda_link2" link2="panda_link6" reason="Never" />
-    <disable_collisions link1="panda_link3" link2="panda_link4" reason="Adjacent" />
-    <disable_collisions link1="panda_link3" link2="panda_link5" reason="Never" />
-    <disable_collisions link1="panda_link3" link2="panda_link6" reason="Never" />
-    <disable_collisions link1="panda_link3" link2="panda_link7" reason="Never" />
-    <disable_collisions link1="panda_link4" link2="panda_link5" reason="Adjacent" />
-    <disable_collisions link1="panda_link4" link2="panda_link6" reason="Never" />
-    <disable_collisions link1="panda_link4" link2="panda_link7" reason="Never" />
-    <disable_collisions link1="panda_link5" link2="panda_link6" reason="Adjacent" />
-    <disable_collisions link1="panda_link6" link2="panda_link7" reason="Adjacent" />
-  </xacro:macro>
-</robot>
+/home/merlabros2/RBE595/src/franka_moveit_config/config/panda_arm.xacro

File: install/franka_moveit_config/share/franka_moveit_config/config/panda_arm_hand.srdf.xacro (robot description, xacro)
@@ -1,43 +1 @@
-<?xml version='1.0' encoding='utf-8'?>
-<!--This does not replace URDF, and is not an extension of URDF.
-    This is a format for representing semantic information about the robot structure.
-    A URDF file must exist for this robot as well, where the joints and the links that are referenced are defined
--->
-<robot xmlns:xacro="http://www.ros.org/wiki/xacro" name="panda">
-  <xacro:include filename="$(find moveit_resources_panda_moveit_config)/config/panda_arm.xacro" />
-  <xacro:include filename="$(find moveit_resources_panda_moveit_config)/config/hand.xacro" />
-  <xacro:panda_arm />
-  <xacro:hand />
-  <!--GROUPS: Representation of a set of joints and links. This can be useful for specifying DOF to plan for, defining arms, end effectors, etc-->
-  <!--LINKS: When a link is specified, the parent joint of that link (if it exists) is automatically included-->
-  <!--JOINTS: When a joint is specified, the child link of that joint (which will always exist) is automatically included-->
-  <!--CHAINS: When a chain is specified, all the links along the chain (including endpoints) are included in the group. Additionally, all the joints that are parents to included links are also included. This means that joints along the chain and the parent joint of the base link are included in the group-->
-  <!--SUBGROUPS: Groups can also be formed by referencing to already defined group names-->
-  <group name="panda_arm_hand">
-    <group name="panda_arm" />
-    <group name="hand" />
-  </group>
-  <group_state name="open" group="hand">
-    <joint name="panda_finger_joint1" value="0.035" />
-    <joint name="panda_finger_joint2" value="0.035" />
-  </group_state>
-  <group_state name="close" group="hand">
-    <joint name="panda_finger_joint1" value="0" />
-    <joint name="panda_finger_joint2" value="0" />
-  </group_state>
-  <!--END EFFECTOR: Purpose: Represent information about an end effector.-->
-  <end_effector name="hand" parent_link="panda_link8" group="hand" parent_group="panda_arm" />
-  <!--DISABLE COLLISIONS: By default it is assumed that any link of the robot could potentially come into collision with any other link in the robot. This tag disables collision checking between a specified pair of links. -->
-  <disable_collisions link1="panda_hand" link2="panda_link3" reason="Never" />
-  <disable_collisions link1="panda_hand" link2="panda_link4" reason="Never" />
-  <disable_collisions link1="panda_hand" link2="panda_link6" reason="Never" />
-  <disable_collisions link1="panda_hand" link2="panda_link7" reason="Adjacent" />
-  <disable_collisions link1="panda_leftfinger" link2="panda_link3" reason="Never" />
-  <disable_collisions link1="panda_leftfinger" link2="panda_link4" reason="Never" />
-  <disable_collisions link1="panda_leftfinger" link2="panda_link6" reason="Never" />
-  <disable_collisions link1="panda_leftfinger" link2="panda_link7" reason="Never" />
-  <disable_collisions link1="panda_link3" link2="panda_rightfinger" reason="Never" />
-  <disable_collisions link1="panda_link4" link2="panda_rightfinger" reason="Never" />
-  <disable_collisions link1="panda_link6" link2="panda_rightfinger" reason="Never" />
-  <disable_collisions link1="panda_link7" link2="panda_rightfinger" reason="Never" />
-</robot>
+/home/merlabros2/RBE595/src/franka_moveit_config/config/panda_arm_hand.srdf.xacro

File: src/franka_moveit_config/config/panda.urdf.xacro (robot description, xacro)
@@ -1,9 +1,12 @@
 <?xml version="1.0"?>
 <robot xmlns:xacro="http://www.ros.org/wiki/xacro" name="panda">
-    <xacro:arg name="initial_positions_file" default="initial_positions.yaml" />
-    <!-- Import panda urdf file -->
-    <xacro:include filename="$(find moveit_resources_panda_description)/urdf/panda.urdf" />
-    <!-- Import control_xacro -->
-    <xacro:include filename="panda.ros2_control.xacro" />
-    <xacro:panda_ros2_control name="FakeSystem" initial_positions_file="$(arg initial_positions_file)"/>
+  <xacro:arg name="initial_positions_file" default="initial_positions.yaml" />
+  <!-- Import the base Panda model -->
+  <xacro:include filename="$(find moveit_resources_panda_description)/urdf/panda.urdf" />
+  <!-- Add ros2_control hardware interface -->
+  <xacro:include filename="$(find franka_description)/urdf/panda.ros2_control.xacro"/>
+  <xacro:panda_ros2_control name="FakeSystem"/>
+  <!-- Add ros2_control for hand -->
+  <xacro:include filename="$(find franka_description)/urdf/panda_hand_control.xacro"/>
+  <xacro:panda_hand_ros2_control name="FakeSystemHand"/>
 </robot>
