Commit message: attempted hardware integration

File: src/franka_description/urdf/panda.ros2_control.xacro (robot description, xacro)
@@ -1,10 +1,15 @@
 <?xml version="1.0"?>
-<robot xmlns:xacro="http://ros.org/wiki/xacro">
-  <!--
-    Minimal ros2_control setup for the Franka arm using FakeSystem.
-    This will simulate joint states & controllers for testing.
-  -->
-  <xacro:macro name="panda_ros2_control" params="name">
-    <ros2_control name="${name}" type="system">
+<!-- ================================================================ -->
+<!--  ROS 2 Control Configuration for Franka Panda Arm (Arm Only)     -->
+<!--  Supports both FakeSystem and Real Hardware Modes                -->
+<!-- ================================================================ -->
+<xacro:macro name="panda_ros2_control"
+             params="name robot_ip:=172.16.0.2 use_fake_hardware:=true"
+             xmlns:xacro="http://www.ros.org/wiki/xacro">
+  <ros2_control name="${name}" type="system">
+    <!-- ============================================================= -->
+    <!--   1. Hardware Selection (Fake vs Real)                        -->
+    <!-- ============================================================= -->
+    <xacro:if value="${use_fake_hardware}">
       <hardware>
         <plugin>fake_components/GenericSystem</plugin>
@@ -12,40 +17,66 @@
         <param name="state_following_offset">0.0</param>
       </hardware>
-      <joint name="panda_joint1">
-        <command_interface name="position"/>
-        <state_interface name="position"/>
-        <state_interface name="velocity"/>
-      </joint>
-      <joint name="panda_joint2">
-        <command_interface name="position"/>
-        <state_interface name="position"/>
-        <state_interface name="velocity"/>
-      </joint>
-      <joint name="panda_joint3">
-        <command_interface name="position"/>
-        <state_interface name="position"/>
-        <state_interface name="velocity"/>
-      </joint>
-      <joint name="panda_joint4">
-        <command_interface name="position"/>
-        <state_interface name="position"/>
-        <state_interface name="velocity"/>
-      </joint>
-      <joint name="panda_joint5">
-        <command_interface name="position"/>
-        <state_interface name="position"/>
-        <state_interface name="velocity"/>
-      </joint>
-      <joint name="panda_joint6">
-        <command_interface name="position"/>
-        <state_interface name="position"/>
-        <state_interface name="velocity"/>
-      </joint>
-      <joint name="panda_joint7">
-        <command_interface name="position"/>
-        <state_interface name="position"/>
-        <state_interface name="velocity"/>
-      </joint>
-    </ros2_control>
-  </xacro:macro>
-</robot>
+    </xacro:if>
+    <xacro:unless value="${use_fake_hardware}">
+      <hardware>
+        <plugin>franka_hardware/FrankaSystemHardware</plugin>
+        <param name="robot_ip">${robot_ip}</param>
+      </hardware>
+    </xacro:unless>
+    <!-- ============================================================= -->
+    <!--   2. Arm Joint Interfaces                                     -->
+    <!-- ============================================================= -->
+    <joint name="panda_joint1">
+      <command_interface name="position"/>
+      <state_interface name="position"/>
+      <state_interface name="velocity"/>
+    </joint>
+    <joint name="panda_joint2">
+      <command_interface name="position"/>
+      <state_interface name="position"/>
+      <state_interface name="velocity"/>
+    </joint>
+    <joint name="panda_joint3">
+      <command_interface name="position"/>
+      <state_interface name="position"/>
+      <state_interface name="velocity"/>
+    </joint>
+    <joint name="panda_joint4">
+      <command_interface name="position"/>
+      <state_interface name="position"/>
+      <state_interface name="velocity"/>
+    </joint>
+    <joint name="panda_joint5">
+      <command_interface name="position"/>
+      <state_interface name="position"/>
+      <state_interface name="velocity"/>
+    </joint>
+    <joint name="panda_joint6">
+      <command_interface name="position"/>
+      <state_interface name="position"/>
+      <state_interface name="velocity"/>
+    </joint>
+    <joint name="panda_joint7">
+      <command_interface name="position"/>
+      <state_interface name="position"/>
+      <state_interface name="velocity"/>
+    </joint>
+    <!-- ============================================================= -->
+    <!--   3. Controller Configuration                                 -->
+    <!-- ============================================================= -->
+    <controller name="panda_arm_controller"
+                type="joint_trajectory_controller/JointTrajectoryController">
+      <joints>
+        panda_joint1
+        panda_joint2
+        panda_joint3
+        panda_joint4
+        panda_joint5
+        panda_joint6
+        panda_joint7
+      </joints>
+      <param name="command_interfaces">["position"]</param>
+      <param name="state_interfaces">["position","velocity"]</param>
+    </controller>
+  </ros2_control>
+</xacro:macro>

File: src/franka_description/urdf/panda_hand_control.xacro (robot description, xacro)
@@ -18,3 +18,2 @@
     </ros2_control>
   </xacro:macro>
-</robot>
